Commit message: problem of orientation difference of PI between end effector and world frame is solved

File: crustcrawler_description/urdf/backup.xacro (robot description, xacro)
@@ -60,5 +60,5 @@
 	        <!-- Arm's base joint -->
 	        <joint name="base_joint" type="fixed">
-	            <origin xyz="0 0 0" rpy="0 0 0" />
+	            <origin xyz="0 0 0" rpy="0 0 ${PI}" />
 	            <parent link="world"/>
 	            <child link="base"/>
@@ -78,13 +78,13 @@
 	        <!-- joint 2 -->
 	        <joint name="joint_2" type="revolute" >
-	            <origin xyz="0 -0.06 0.06" rpy="0 0 0" />
+	            <origin xyz="0 -0.06 0.06" rpy="${PI/2} 0 0" />
 	            <parent link="link_joint_2" />
 	            <child link="connector_1"/>
-	            <axis xyz="0 1 0"/>
+	            <axis xyz="0 0 1"/>
 	            <limit  lower="-1.6" upper="1.6" effort="15" velocity="1.7" />
 	        </joint>
 	        <!-- Fixed joint between connector_1 and the first girder -->
 	        <joint name="connector_1_girder_1_joint" type="fixed">
-	            <origin xyz="-0.0153 0.06 0.036" rpy="0 0 0" />
+	            <origin xyz="-0.0153 0.036 -0.06" rpy="-${PI/2} 0 0" />
 	            <parent link="connector_1"/>
 	            <child link="link_girder_1"/>
@@ -101,5 +101,5 @@
 	            <parent link="link_joint_3" />
 	            <child link="connector_2"/>
-	            <axis xyz="0 -1 0"/>
+	            <axis xyz="0 1 0"/>
 	            <limit  lower="-1.9" upper="1.9" effort="8.4" velocity="1.7" />
 	        </joint>
@@ -112,5 +112,5 @@
 	        <!-- Fixed joint between second girder joint_4 -->
 	        <joint name="girder_2_joint_4_joint" type="fixed">
-	            <origin xyz="0.0153 0 0.0635" rpy="0 0 ${PI}" />
+	            <origin xyz="0.0153 0 0.0635" rpy="0 0 0" />
 	            <parent link="link_girder_2"/>
 	            <child link="link_joint_4"/>
@@ -165,5 +165,5 @@
 	        </joint>
 	        <joint name="crustcrawler_endpoint" type="fixed">
-	      <origin rpy="0 0 ${PI}" xyz="0 0 0.13"/>
+	      <origin rpy="0 0 0" xyz="0 0 0.13"/>
 	      <parent link="link_gripper_base"/>
 	      <child link="the_gripper"/>
@@ -216,5 +216,5 @@
 	        <link name="connector_1">
 	            <visual>
-	                <origin xyz="0 0.06 0" rpy="0 0 0" />
+	                <origin xyz="0 0 -0.06" rpy="-${PI/2} 0 0" />
 	                <geometry>
 	                    <mesh filename="package://crustcrawler_description/meshes/collada/connecter_joint_2_girder_1.dae"/>
