Commit message: modified urdfs for approximate mass and inertia tensors

File: crustcrawler_description/urdf/crustcrawler_arm_high_speed.xacro (robot description, xacro)
@@ -69,5 +69,5 @@
             <child link="link_joint_2"/>
             <axis xyz="0 0 1"/>
-            <limit  lower="-1.8" upper="2.3" effort="6.0" velocity="1.7" />
+            <limit  lower="-1.8" upper="2.3" effort="6.0" velocity="2.4" />
         </joint>
         <!-- joint 2 -->
@@ -77,5 +77,5 @@
             <child link="connector_1"/>
             <axis xyz="0 1 0"/>
-            <limit  lower="-1.6" upper="1.6" effort="15" velocity="1.7" />
+            <limit  lower="-1.6" upper="1.6" effort="15" velocity="2.4" />
         </joint>
         <!-- Fixed joint between connector_1 and the first girder -->
@@ -97,5 +97,5 @@
             <child link="connector_2"/>
             <axis xyz="0 1 0"/>
-            <limit  lower="-1.9" upper="1.9" effort="8.4" velocity="1.7" />
+            <limit  lower="-1.9" upper="1.9" effort="8.4" velocity="2.4" />
         </joint>
         <!-- Fixed joint between connector_2 and link_girder_2 -->
@@ -117,5 +117,5 @@
             <child link="link_joint_5"/>
             <axis xyz="0 0 1"/>
-            <limit  lower="-3.14" upper="3.14" effort="6.0" velocity="1.7" />
+            <limit  lower="-3.0" upper="3.0" effort="6.0" velocity="2.4" />
         </joint>
         <!-- joint 5 -->
@@ -125,5 +125,5 @@
             <child link="connector_3"/>
             <axis xyz="0 1 0"/>
-            <limit  lower="-1.6" upper="1.6" effort="2.5" velocity="1.7" />
+            <limit  lower="-1.6" upper="1.6" effort="2.5" velocity="2.4" />
         </joint>
         <!-- Fixed joint between connector_3 and joint_6 -->
@@ -139,5 +139,5 @@
             <child link="link_gripper_base"/>
             <axis xyz="0 0 1"/>
-            <limit  lower="-3.140" upper="3.140" effort="2.5" velocity="1.7" />
+            <limit  lower="-3.0" upper="3.0" effort="2.5" velocity="2.4" />
         </joint>
         <!-- Gripper right finger joint -->
@@ -148,5 +148,5 @@
             <axis xyz="1 0 0"/>
             <!-- From 14 to -45 degrees -->
-            <limit  lower="-0.84" upper="0.84" effort="1.8" velocity="1.7" />
+            <limit  lower="-0.84" upper="0.84" effort="1.8" velocity="2.4" />
         </joint>
         <!-- Gripper left finger joint -->
@@ -157,5 +157,5 @@
             <axis xyz="1 0 0"/>
             <!-- From 14 to -45 degrees -->
-            <limit  lower="-0.84" upper="0.84" effort="1.8" velocity="1.7" />
+            <limit  lower="-0.84" upper="0.84" effort="1.8" velocity="2.4" />
         </joint>
         <joint name="crustcrawler_endpoint" type="fixed">

Commit message: modified controller node for throwing ball into a box

File: crustcrawler_description/urdf/crustcrawler_arm_high_speed.xacro (robot description, xacro)
@@ -69,5 +69,5 @@
             <child link="link_joint_2"/>
             <axis xyz="0 0 1"/>
-            <limit  lower="-1.8" upper="2.3" effort="6.0" velocity="2.4" />
+            <limit  lower="-1.8" upper="2.3" effort="6.0" velocity="2.0" />
         </joint>
         <!-- joint 2 -->
@@ -77,5 +77,5 @@
             <child link="connector_1"/>
             <axis xyz="0 1 0"/>
-            <limit  lower="-1.6" upper="1.6" effort="15" velocity="2.4" />
+            <limit  lower="-1.6" upper="1.6" effort="15" velocity="2.0" />
         </joint>
         <!-- Fixed joint between connector_1 and the first girder -->
@@ -97,5 +97,5 @@
             <child link="connector_2"/>
             <axis xyz="0 1 0"/>
-            <limit  lower="-1.9" upper="1.9" effort="8.4" velocity="2.4" />
+            <limit  lower="-1.9" upper="1.9" effort="8.4" velocity="2.0" />
         </joint>
         <!-- Fixed joint between connector_2 and link_girder_2 -->
@@ -117,5 +117,5 @@
             <child link="link_joint_5"/>
             <axis xyz="0 0 1"/>
-            <limit  lower="-3.0" upper="3.0" effort="6.0" velocity="2.4" />
+            <limit  lower="-3.0" upper="3.0" effort="6.0" velocity="2.0" />
         </joint>
         <!-- joint 5 -->
@@ -125,5 +125,5 @@
             <child link="connector_3"/>
             <axis xyz="0 1 0"/>
-            <limit  lower="-1.6" upper="1.6" effort="2.5" velocity="2.4" />
+            <limit  lower="-1.6" upper="1.6" effort="2.5" velocity="2.0" />
         </joint>
         <!-- Fixed joint between connector_3 and joint_6 -->
@@ -139,5 +139,5 @@
             <child link="link_gripper_base"/>
             <axis xyz="0 0 1"/>
-            <limit  lower="-3.0" upper="3.0" effort="2.5" velocity="2.4" />
+            <limit  lower="-3.0" upper="3.0" effort="2.5" velocity="2.0" />
         </joint>
         <!-- Gripper right finger joint -->
@@ -148,5 +148,5 @@
             <axis xyz="1 0 0"/>
             <!-- From 14 to -45 degrees -->
-            <limit  lower="-0.84" upper="0.84" effort="1.8" velocity="2.4" />
+            <limit  lower="-0.84" upper="0.84" effort="1.8" velocity="2.0" />
         </joint>
         <!-- Gripper left finger joint -->
@@ -157,5 +157,5 @@
             <axis xyz="1 0 0"/>
             <!-- From 14 to -45 degrees -->
-            <limit  lower="-0.84" upper="0.84" effort="1.8" velocity="2.4" />
+            <limit  lower="-0.84" upper="0.84" effort="1.8" velocity="2.0" />
         </joint>
         <joint name="crustcrawler_endpoint" type="fixed">

Commit message: last version with frames orientations corrected in the simulated version, to be tested with the real robot

File: crustcrawler_description/urdf/crustcrawler_arm_high_speed.xacro (robot description, xacro)
@@ -59,5 +59,4 @@
         <!-- Arm's base joint -->
         <joint name="arm_base_joint" type="fixed">
-            <origin xyz="0 0 0" rpy="0 0 ${PI}" />
             <parent link="world"/>
             <child link="link_joint_1"/>

File: crustcrawler_description/urdf/crustcrawler_arm_test_2.xacro (robot description, xacro)
@@ -59,5 +59,4 @@
         <!-- Arm's base joint -->
         <joint name="arm_base_joint" type="fixed">
-            <origin xyz="0 0 0" rpy="0 0 ${PI}" />
             <parent link="world"/>
             <child link="link_joint_1"/>

File: crustcrawler_description/urdf/crustcrawler_kinect.urdf.xacro (robot description, xacro)
@@ -4,5 +4,5 @@
    <joint name="camera_rgb_joint" type="fixed">
       <!--origin xyz="1.8 0.4 0.4" rpy="0 0.5 -3.14"/-->
-      <origin xyz="0.85 -0.225 0.813" rpy="-0.124 0.77 2.94"/>
+      <origin xyz="1.5 -0.225 0.813" rpy="-0.124 0.77 2.94"/>
       <parent link="world"/>
       <child link="camera_rgb_frame" />

Commit message: correcting other description URDFs and the STL files

File: crustcrawler_description/urdf/crustcrawler_arm_high_speed.xacro (robot description, xacro)
@@ -50,4 +50,5 @@
         <!-- ****** JOINT DEFINITIONS ****** -->
         <link name="world"/>
+		<link name="base"/>
         <link name="the_gripper">
       <inertial>
@@ -58,8 +59,13 @@
     </link>
         <!-- Arm's base joint -->
-        <joint name="arm_base_joint" type="fixed">
-            <parent link="world"/>
-            <child link="link_joint_1"/>
-        </joint>
+	        <joint name="base_joint" type="fixed">
+	            <origin xyz="0 0 0" rpy="0 0 0" />
+	            <parent link="world"/>
+	            <child link="base"/>
+	        </joint>
+	        <joint name="arm_base_joint" type="fixed">
+	            <parent link="base"/>
+	            <child link="link_joint_1"/>
+	        </joint>
         <!-- joint 1 -->
         <joint name="joint_1" type="revolute" >
@@ -95,5 +101,5 @@
             <parent link="link_joint_3" />
             <child link="connector_2"/>
-            <axis xyz="0 1 0"/>
+            <axis xyz="0 -1 0"/>
             <limit  lower="-1.9" upper="1.9" effort="8.4" velocity="2.0" />
         </joint>
@@ -123,5 +129,5 @@
             <parent link="link_joint_5" />
             <child link="connector_3"/>
-            <axis xyz="0 1 0"/>
+            <axis xyz="0 -1 0"/>
             <limit  lower="-1.6" upper="1.6" effort="2.5" velocity="2.0" />
         </joint>
