Commit message: latest version

File: crustcrawler_description/urdf/crustcrawler_kinect.urdf.xacro (robot description, xacro)
@@ -3,7 +3,6 @@
   <!-- kinect with all frames as defined in turtlebot -->
    <joint name="camera_rgb_joint" type="fixed">
-      <!--origin xyz="1.8 0.4 0.4" rpy="0 0.5 -3.14"/-->
-      <origin xyz="1.5 -0.225 0.813" rpy="-0.124 0.77 2.94"/>
-      <parent link="world"/>
+      <origin xyz="0 -0.045 0" rpy="0 0 0"/>
+      <parent link="camera_link"/>
       <child link="camera_rgb_frame" />
   </joint>
@@ -16,6 +15,6 @@
   <link name="camera_rgb_optical_frame"/>
   <joint name="kinect_joint" type="fixed">
-      <origin xyz="0 0 0" rpy="0 0 1.5707963267948966"/>
-      <parent link="camera_rgb_frame"/>
+      <origin xyz="1.5 0.0 0.813" rpy="0 0.77 3.14"/>
+      <parent link="base"/>
       <child link="camera_link"/>
   </joint>
@@ -24,13 +23,13 @@
        <origin xyz="0 0 0" rpy="0 0 0"/>
         <geometry>
-         <mesh filename="package://baxter_description/meshes/sensors/kinect.dae"/>
+         <mesh filename="package://crustcrawler_description/meshes/sensors/kinect.dae"/>
         </geometry>
       </visual>
-  	  <collision>
-        <origin xyz="0.0 0.0 0.0" rpy="0 0 0"/>
-  	    <geometry>
-  	      <box size="0.07271 0.27794 0.073"/>
-  	    </geometry>
-  	  </collision>
+      <collision>
+        <origin xyz="0 0 0" rpy="0 0 0"/>
+        <geometry>
+          <box size="0.07271 0.27794 0.073"/>
+        </geometry>
+      </collision>
       <inertial>
         <mass value="0.564" />
@@ -45,24 +44,17 @@
          (Hence, don't publish them additionally!) -->
   <joint name="camera_depth_joint" type="fixed">
-	  <origin xyz="0 0.025 0" rpy="0 0 0" />
-	  <parent link="camera_rgb_frame" />
-	  <child link="camera_depth_frame" />
+    <origin xyz="0 0.025 0" rpy="0 0 0" />
+    <parent link="camera_rgb_frame" />
+    <child link="camera_depth_frame" />
   </joint>
   <link name="camera_depth_frame"/>
-	<joint name="camera_depth_optical_joint" type="fixed">
-	  <origin xyz="0 0 0" rpy="-1.5707963267948966 0 -1.5707963267948966" />
-	  <parent link="camera_depth_frame" />
-	  <child link="camera_depth_optical_frame" />
-	</joint>
-	<link name="camera_depth_optical_frame"/>
-<!-- ros_control plugin -->
-  <!--gazebo>
-    <plugin name="gazebo_ros_control" filename="libgazebo_ros_control.so">
-      <robotNamespace>/baxter</robotNamespace>
-      <robotSimType>gazebo_ros_control/DefaultRobotHWSim</robotSimType>
-    </plugin>
-  </gazebo-->
+  <joint name="camera_depth_optical_joint" type="fixed">
+    <origin xyz="0 0 0" rpy="-1.5707963267948966 0 -1.5707963267948966" />
+    <parent link="camera_depth_frame" />
+    <child link="camera_depth_optical_frame" />
+  </joint>
+  <link name="camera_depth_optical_frame"/>
 <!-- Microsoft Kinect / ASUS Xtion PRO Live for simulation -->
-    <gazebo reference="camera_rgb_frame">
+    <gazebo reference="camera_link">
       <sensor type="depth" name="camera">
         <always_on>true</always_on>
@@ -76,29 +68,34 @@
           </image>
           <clip>
-            <near>0.9</near>
+            <near>0.05</near>
             <far>8.0</far>
           </clip>
         </camera>
         <plugin name="kinect_camera_controller" filename="libgazebo_ros_openni_kinect.so">
-          <cameraName>camera</cameraName>
+          <baseline>0.2</baseline>
           <alwaysOn>true</alwaysOn>
           <updateRate>10</updateRate>
+          <cameraName>camera</cameraName>
           <imageTopicName>rgb/image_rect_color</imageTopicName>
           <depthImageTopicName>depth_registered/sw_registered/image_rect</depthImageTopicName>
-          <pointCloudTopicName>depth_registered/points</pointCloudTopicName>
+          <pointCloudTopicName>depth_registered/sw_registered/points</pointCloudTopicName>
           <cameraInfoTopicName>rgb/camera_info</cameraInfoTopicName>
           <depthImageCameraInfoTopicName>depth_registered/sw_registered/camera_info</depthImageCameraInfoTopicName>
           <frameName>camera_depth_optical_frame</frameName>
-          <baseline>0.1</baseline>
-          <distortion_k1>0.0</distortion_k1>
-          <distortion_k2>0.0</distortion_k2>
-          <distortion_k3>0.0</distortion_k3>
-          <distortion_t1>0.0</distortion_t1>
-          <distortion_t2>0.0</distortion_t2>
-          <pointCloudCutoff>0.4</pointCloudCutoff>
+          <pointCloudCutoff>0.5</pointCloudCutoff>
+          <distortionK1>0.00000001</distortionK1>
+          <distortionK2>0.00000001</distortionK2>
+          <distortionK3>0.00000001</distortionK3>
+          <distortionT1>0.00000001</distortionT1>
+          <distortionT2>0.00000001</distortionT2>
+          <CxPrime>0</CxPrime>
+          <Cx>0</Cx>
+          <Cy>0</Cy>
+          <focalLength>0</focalLength>
+          <hackBaseline>0</hackBaseline>
         </plugin>
       </sensor>
     </gazebo>
-  <!-- Baxter Base URDF -->
+  <!-- Crustcrawler Base URDF -->
   <xacro:include filename="$(find crustcrawler_description)/urdf/crustcrawler_arm_test_2.xacro"/>
 </robot>

Commit message: working version with pick and place, with or without camera kinect2

File: crustcrawler_description/urdf/crustcrawler_kinect.urdf.xacro (robot description, xacro)
@@ -3,5 +3,5 @@
   <!-- kinect with all frames as defined in turtlebot -->
    <joint name="camera_rgb_joint" type="fixed">
-      <origin xyz="0 -0.045 0" rpy="0 0 0"/>
+      <origin xyz="0 0.0 0" rpy="0 0 0"/>
       <parent link="camera_link"/>
       <child link="camera_rgb_frame" />
@@ -44,5 +44,5 @@
          (Hence, don't publish them additionally!) -->
   <joint name="camera_depth_joint" type="fixed">
-    <origin xyz="0 0.025 0" rpy="0 0 0" />
+    <origin xyz="0 0.0 0" rpy="0 0 0" />
     <parent link="camera_rgb_frame" />
     <child link="camera_depth_frame" />
