Commit message: latest version on crustcrawler laptop

File: crustcrawler_description/urdf/crustcrawler_arm_test_2.xacro (robot description, xacro)
@@ -74,5 +74,5 @@
 	            <child link="link_joint_2"/>
 	            <axis xyz="0 0 1"/>
-	            <limit  lower="-1.8" upper="2.3" effort="6.0" velocity="1.7" />
+	            <limit  lower="-1.8" upper="2.3" effort="6.0" velocity="2.0" />
 	        </joint>
 	        <!-- joint 2 -->
@@ -82,5 +82,5 @@
 	            <child link="connector_1"/>
 	            <axis xyz="0 1 0"/>
-	            <limit  lower="-1.6" upper="1.6" effort="15" velocity="1.7" />
+	            <limit  lower="-1.6" upper="1.6" effort="15" velocity="2.0" />
 	        </joint>
 	        <!-- Fixed joint between connector_1 and the first girder -->
@@ -102,5 +102,5 @@
 	            <child link="connector_2"/>
 	            <axis xyz="0 -1 0"/>
-	            <limit  lower="-1.9" upper="1.9" effort="8.4" velocity="1.7" />
+	            <limit  lower="-1.9" upper="1.9" effort="8.4" velocity="2.0" />
 	        </joint>
 	        <!-- Fixed joint between connector_2 and link_girder_2 -->
@@ -122,5 +122,5 @@
 	            <child link="link_joint_5"/>
 	            <axis xyz="0 0 1"/>
-	            <limit  lower="-3.14" upper="3.14" effort="6.0" velocity="1.7" />
+	            <limit  lower="-3.14" upper="3.14" effort="6.0" velocity="2.0" />
 	        </joint>
 	        <!-- joint 5 -->
@@ -130,5 +130,5 @@
 	            <child link="connector_3"/>
 	            <axis xyz="0 -1 0"/>
-	            <limit  lower="-1.6" upper="1.6" effort="2.5" velocity="1.7" />
+	            <limit  lower="-1.6" upper="1.6" effort="2.5" velocity="2.0" />
 	        </joint>
 	        <!-- Fixed joint between connector_3 and joint_6 -->
@@ -144,5 +144,5 @@
 	            <child link="link_gripper_base"/>
 	            <axis xyz="0 0 1"/>
-	            <limit  lower="-3.140" upper="3.140" effort="2.5" velocity="1.7" />
+	            <limit  lower="-3.140" upper="3.140" effort="2.5" velocity="2.0" />
 	        </joint>
 	        <!-- Gripper right finger joint -->
@@ -153,5 +153,5 @@
 	            <axis xyz="1 0 0"/>
 	            <!-- From 14 to -45 degrees -->
-	            <limit  lower="-0.84" upper="0.84" effort="1.8" velocity="1.7" />
+	            <limit  lower="-0.84" upper="0.84" effort="1.8" velocity="2.0" />
 	        </joint>
 	        <!-- Gripper left finger joint -->
@@ -162,5 +162,5 @@
 	            <axis xyz="1 0 0"/>
 	            <!-- From 14 to -45 degrees -->
-	            <limit  lower="-0.84" upper="0.84" effort="1.8" velocity="1.7" />
+	            <limit  lower="-0.84" upper="0.84" effort="1.8" velocity="2.0" />
 	        </joint>
 	        <joint name="crustcrawler_endpoint" type="fixed">

Commit message: latest version working with babbling and pick and place application on the crustcrawler laptop

File: crustcrawler_description/urdf/crustcrawler_arm_test_2.xacro (robot description, xacro)
@@ -165,5 +165,5 @@
 	        </joint>
 	        <joint name="crustcrawler_endpoint" type="fixed">
-	      <origin rpy="0 0 0" xyz="0 0 0.16"/>
+	      <origin rpy="0 0 0" xyz="0 0 0.18"/>
 	      <parent link="link_gripper_base"/>
 	      <child link="the_gripper"/>

Commit message: latest version on the main laptop

File: crustcrawler_description/urdf/crustcrawler_arm_test_2.xacro (robot description, xacro)
@@ -165,5 +165,5 @@
 	        </joint>
 	        <joint name="crustcrawler_endpoint" type="fixed">
-	      <origin rpy="0 0 0" xyz="0 0 0.16"/>
+	      <origin rpy="0 0 0" xyz="0 0 0.13"/>
 	      <parent link="link_gripper_base"/>
 	      <child link="the_gripper"/>

Commit message: changes for some topics in moveit_grasping to work with a name space prefix, also some changes to the urdf

File: crustcrawler_description/urdf/crustcrawler_arm_test_2.xacro (robot description, xacro)
@@ -165,5 +165,5 @@
 	        </joint>
 	        <joint name="crustcrawler_endpoint" type="fixed">
-	      <origin rpy="0 0 0" xyz="0 0 0.13"/>
+	      <origin rpy="0 0 0" xyz="0 0 0.17"/>
 	      <parent link="link_gripper_base"/>
 	      <child link="the_gripper"/>
